File: LDR_pai.kicad_pcb (KiCad board)
At the start: 2 copper layers, 70 x 40 mm, 19 parts, among them J1 Screw_Terminal_01x04, J2 Screw_Terminal_01x02, K1 FINDER-36.11, U1 LM555xN

Commit message: data refresh
Parts:
- removed R2: LDR07, OptoDevice:R_LDR_5.1x4.3mm_P3.4mm_Vertical
- JP1: footprint TestPoint:TestPoint_2Pads_Pitch5.08mm_Drill1.3mm -> TestPoint:TestPoint_2Pads_Pitch2.54mm_Drill0.8mm
- moved JP1 31.6 mm to (117.4, 59.8), turned to 90 degrees
- moved C1 1.41 mm to (112.9, 74.0)
Connections:
- net /Timer_Trigger renamed /LDR_1
- J1 pad 1: VCC -> +12V
Routing:
- net /LDR_1: track 0.00 -> 136.1 mm
- net +12V: track 0.00 -> 111.4 mm, vias 0 -> 2
- net /Timer_Output: track 0.00 -> 68.5 mm, vias 0 -> 2
- net Net-(R1-Pad1): track 0.00 -> 50.6 mm, vias 0 -> 2
- net Net-(C2-Pad1): track 0.00 -> 49.9 mm, vias 0 -> 2
- net Net-(C1-Pad1): track 0.00 -> 44.0 mm
- net Net-(R3-Pad1): track 0.00 -> 31.0 mm, vias 0 -> 2
- net /R_out: track 0.00 -> 29.5 mm
- net /R_in: track 0.00 -> 20.2 mm
- net Net-(D3-Pad2): track 0.00 -> 18.1 mm
- net GND: track 0.00 -> 14.8 mm, vias 0 -> 2
- net Net-(C4-Pad1): track 0.00 -> 10.6 mm
- net Net-(D2-Pad1): track 0.00 -> 9.39 mm
- added copper zone on F.Cu, net GND
Other:
- board size 70 x 40 mm -> 71 x 41.6 mm
- board text added: "Cinza"
- board text added: "Fio unico com curvas"
- board text added: "Laranja"
