File: LDR_pai.kicad_sch (KiCad schematic)
At the start: 19 parts, among them J1 Screw_Terminal_01x04, J2 Screw_Terminal_01x02, K1 FINDER-36.11, U1 LM555xN

Commit message: data refresh
Parts:
- JP1: footprint TestPoint:TestPoint_2Pads_Pitch5.08mm_Drill1.3mm -> TestPoint:TestPoint_2Pads_Pitch2.54mm_Drill0.8mm
- R2: now left out of the parts list
Connections:
- net VCC is gone; now on net +12V: J1.1 (Pin_1)
- net GND: no longer R2.2
- net LDR_1: no longer R2.1
Changed lines of the file:
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@@
   (junction (at 127.635 76.2) (diameter 0) (color 0 0 0 0)
   )
-  (junction (at 40.64 135.89) (diameter 0) (color 0 0 0 0)
-  )
   (junction (at 127.635 94.615) (diameter 0) (color 0 0 0 0)
   )
@@
     (stroke (width 0) (type default) (color 0 0 0 0))
   )
-  (wire (pts (xy 45.085 133.35) (xy 45.085 135.89))
-    (stroke (width 0) (type default) (color 0 0 0 0))
-  )
   (wire (pts (xy 74.295 120.015) (xy 74.295 127))
     (stroke (width 0) (type default) (color 0 0 0 0))
@@
     (stroke (width 0) (type default) (color 0 0 0 0))
   )
+  (wire (pts (xy 44.45 127.635) (xy 45.72 130.81))
+    (stroke (width 0) (type default) (color 0 0 0 0))
+  )
   (wire (pts (xy 88.9 137.795) (xy 88.9 132.715))
     (stroke (width 0) (type default) (color 0 0 0 0))
@@
     (stroke (width 0) (type default) (color 0 0 0 0))
   )
-  (wire (pts (xy 45.085 130.81) (xy 45.085 128.27))
-    (stroke (width 0) (type default) (color 0 0 0 0))
-  )
   (wire (pts (xy 109.22 151.13) (xy 112.395 151.13))
     (stroke (width 0) (type default) (color 0 0 0 0))
@@
     (stroke (width 0) (type default) (color 0 0 0 0))
   )
-  (wire (pts (xy 45.72 130.81) (xy 45.085 130.81))
-    (stroke (width 0) (type default) (color 0 0 0 0))
-  )
-  (wire (pts (xy 41.275 106.045) (xy 41.275 108.585))
+  (wire (pts (xy 41.275 104.775) (xy 41.275 108.585))
     (stroke (width 0) (type default) (color 0 0 0 0))
   )
@@
     (stroke (width 0) (type default) (color 0 0 0 0))
   )
-  (wire (pts (xy 40.64 135.89) (xy 40.64 136.525))
-    (stroke (width 0) (type default) (color 0 0 0 0))
-  )
-  (wire (pts (xy 45.085 135.89) (xy 40.64 135.89))
-    (stroke (width 0) (type default) (color 0 0 0 0))
-  )
-  (wire (pts (xy 45.72 133.35) (xy 45.085 133.35))
-    (stroke (width 0) (type default) (color 0 0 0 0))
-  )
   (wire (pts (xy 99.06 148.59) (xy 99.06 149.86))
     (stroke (width 0) (type default) (color 0 0 0 0))
@@
     (stroke (width 0) (type default) (color 0 0 0 0))
   )
-  (wire (pts (xy 45.085 128.27) (xy 40.64 128.27))
-    (stroke (width 0) (type default) (color 0 0 0 0))
-  )
   (wire (pts (xy 40.005 118.11) (xy 43.18 113.665))
     (stroke (width 0) (type default) (color 0 0 0 0))
@@
   )
   (wire (pts (xy 74.295 127) (xy 74.295 129.54))
+    (stroke (width 0) (type default) (color 0 0 0 0))
+  )
+  (wire (pts (xy 44.45 133.35) (xy 45.72 133.35))
+    (stroke (width 0) (type default) (color 0 0 0 0))
+  )
+  (wire (pts (xy 44.45 138.43) (xy 44.45 133.35))
     (stroke (width 0) (type default) (color 0 0 0 0))
   )
@@
     (effects (font (size 1.27 1.27)) (justify left bottom))
   )
-  (label "LDR_1" (at 40.64 128.27 180)
+  (label "LDR_1" (at 44.45 127.635 180)
     (effects (font (size 1.27 1.27)) (justify right bottom))
   )
@@
     (effects (font (size 1.27 1.27)) (justify right bottom))
   )
-  (label "LDR_2" (at 40.64 136.525 270)
+  (label "LDR_2" (at 44.45 138.43 180)
     (effects (font (size 1.27 1.27)) (justify right bottom))
   )
@@
     (effects (font (size 1.27 1.27)) (justify right bottom))
   )
-  (label "12V" (at 41.275 108.585 180)
-    (effects (font (size 1.27 1.27)) (justify right bottom))
-  )
   (symbol (lib_id "Connector:Screw_Terminal_01x02") (at 50.8 130.81 0) (unit 1)
     (in_bom yes) (on_board yes) (fields_autoplaced)
@@
   )
   (symbol (lib_id "Sensor_Optical:LDR07") (at 40.64 132.08 0) (unit 1)
-    (in_bom yes) (on_board yes)
+    (in_bom no) (on_board no)
     (property "Reference" "R2" (id 0) (at 33.655 132.08 0)
       (effects (font (size 1.27 1.27)) (justify left))
@@
     (pin "1")
     (pin "2")
+  )
+  (symbol (lib_id "power:+12V") (at 41.275 104.775 0) (unit 1)
+    (in_bom yes) (on_board yes)
+    (property "Reference" "#PWR?" (id 0) (at 41.275 108.585 0)
+      (effects (font (size 1.27 1.27)) hide)
+    )
+    (property "Value" "+12V" (id 1) (at 38.1 105.41 0))
+    (property "Footprint" "" (id 2) (at 41.275 104.775 0)
+      (effects (font (size 1.27 1.27)) hide)
+    )
+    (property "Datasheet" "" (id 3) (at 41.275 104.775 0)
+      (effects (font (size 1.27 1.27)) hide)
+    )
+    (pin "1")
   )
   (symbol (lib_id "power:+12V") (at 71.755 59.055 0) (unit 1)
@@
       (effects (font (size 1.27 1.27)) hide)
     )
-    (property "Footprint" "TestPoint:TestPoint_2Pads_Pitch5.08mm_Drill1.3mm" (id 2) (at 135.89 94.615 0)
+    (property "Footprint" "TestPoint:TestPoint_2Pads_Pitch2.54mm_Drill0.8mm" (id 2) (at 135.89 94.615 0)
       (effects (font (size 1.27 1.27)) hide)
     )
@@
     (pin "2")
   )
-  (symbol (lib_id "power:VCC") (at 41.275 106.045 0) (unit 1)
-    (in_bom yes) (on_board yes)
-    (property "Reference" "#PWR02" (id 0) (at 41.275 109.855 0)
-      (effects (font (size 1.27 1.27)) hide)
-    )
-    (property "Value" "VCC" (id 1) (at 40.005 102.235 0)
-      (effects (font (size 1.27 1.27)) hide)
-    )
-    (property "Footprint" "" (id 2) (at 41.275 106.045 0)
-      (effects (font (size 1.27 1.27)) hide)
-    )
-    (property "Datasheet" "" (id 3) (at 41.275 106.045 0)
-      (effects (font (size 1.27 1.27)) hide)
-    )
-    (pin "1")
-  )
   (symbol (lib_id "power:+12V") (at 105.41 77.47 0) (unit 1)
     (in_bom yes) (on_board yes)
@@
       (reference "#PWR01") (unit 1) (value "GND") (footprint "")
     )
-    (path "/faf9583a-15f4-490d-aaf8-5442b42418f2"
-      (reference "#PWR02") (unit 1) (value "VCC") (footprint "")
-    )
     (path "/270408a2-7c39-4dd0-9696-8fa401b45e27"
       (reference "#PWR03") (unit 1) (value "+12V") (footprint "")
@@
       (reference "#PWR014") (unit 1) (value "GND") (footprint "")
     )
+    (path "/1f8fbf0b-b135-4bca-a2c3-beacad53b0f0"
+      (reference "#PWR?") (unit 1) (value "+12V") (footprint "")
+    )
     (path "/4abd4be8-4657-44ea-ac20-5794a642d45d"
       (reference "C1") (unit 1) (value "10nF") (footprint "Capacitor_THT:C_Radial_D5.0mm_H5.0mm_P2.00mm")
@@
     )
     (path "/69fee2b6-79d2-4e30-8f1d-940d76f81724"
-      (reference "JP1") (unit 1) (value "Jumper_2_Open") (footprint "TestPoint:TestPoint_2Pads_Pitch5.08mm_Drill1.3mm")
+      (reference "JP1") (unit 1) (value "Jumper_2_Open") (footprint "TestPoint:TestPoint_2Pads_Pitch2.54mm_Drill0.8mm")
     )
     (path "/a8869d14-c275-4004-9be7-de4e15f57b37"
